File: V2.x/Servo/LOCO-Servo.brd (EAGLE design)
At the start: 43.2 x 34.3 mm, 49 parts, among them IC1 Atmega 328-P, IC2 MCP2515, IC3 LM340MP-05, Q1 8MHz, Q2 16MHz, X2 2X6-A

Commit message: design clean up
Changed lines of the file:
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@@
 <hole x="40.64" y="31.75" drill="3.048"/>
 <text x="11.2395" y="31.59125" size="1.27" layer="26" rot="MR0">Servo</text>
-<text x="27.94" y="6.985" size="1.778" layer="25">1</text>
+<text x="25.7175" y="0.79375" size="1.778" layer="25">1</text>
 <text x="11.27125" y="30.1625" size="0.8128" layer="26" rot="MR0">V2.2</text>
 <rectangle x1="12.0777" y1="27.5717" x2="12.2047" y2="27.5971" layer="26" grouprefs="LOCO"/>
@@
 <wire x1="23.92963125" y1="19.05" x2="27.78125" y2="19.05" width="0.1524" layer="26"/>
 <text x="6.0325" y="1.27" size="0.8128" layer="25" rot="R90">GND</text>
-<text x="18.415" y="33.17875" size="0.8128" layer="25" rot="R180" align="center">loco-can.github.io</text>
+<text x="13.0175" y="33.17875" size="0.8128" layer="25" rot="R180" align="center">loco-can.github.io</text>
 </plain>
 <attributes>
@@
 <attribute name="MF" value="" x="-6.35" y="-40.64" size="1.778" layer="27" rot="R270" display="off"/>
 <attribute name="MPN" value="" x="-6.35" y="-40.64" size="1.778" layer="27" rot="R270" display="off"/>
-<attribute name="NAME" x="24.765" y="5.842" size="1.27" layer="25" ratio="10"/>
+<attribute name="NAME" x="21.30425" y="3.175" size="0.8128" layer="25" ratio="10" rot="R90"/>
 <attribute name="OC_FARNELL" value="1667008" x="-6.35" y="-40.64" size="1.778" layer="27" rot="R270" display="off"/>
 <attribute name="OC_NEWARK" value="unknown" x="-6.35" y="-40.64" size="1.778" layer="27" rot="R270" display="off"/>
@@
 </element>
 <element name="IC2" library="mcp2514" package="TSSOP20" value="MCP2515" x="17.145" y="17.145" smashed="yes" rot="R90"/>
-<element name="IC1" library="atmel" library_urn="urn:adsk.eagle:library:105" package="TQFP32-08" package3d_urn="urn:adsk.eagle:package:4313/2" value="Atmega 328-P" x="17.78" y="17.4625" smashed="yes" rot="MR180">
-<attribute name="MF" value="" x="17.78" y="17.4625" size="1.778" layer="28" rot="MR180" display="off"/>
-<attribute name="MPN" value="ATMEGA8-16AU" x="17.78" y="17.4625" size="1.778" layer="28" rot="MR180" display="off"/>
+<element name="IC1" library="atmel" library_urn="urn:adsk.wipprod:fs.file:vf.5DA8-qxERB6VD-tqpl9Cbg" package="TQFP32-08" package3d_urn="urn:adsk.wipprod:fs.file:vf.4VkE7R9WQkCoTiDjtEgskA?version=3" value="Atmega 328-P" x="17.78" y="17.4625" smashed="yes" rot="MR180">
 <attribute name="NAME" x="21.59" y="13.5001" size="0.8128" layer="26" ratio="10" rot="MR180"/>
-<attribute name="OC_FARNELL" value="9171371" x="17.78" y="17.4625" size="1.778" layer="28" rot="MR180" display="off"/>
-<attribute name="OC_NEWARK" value="73M8863" x="17.78" y="17.4625" size="1.778" layer="28" rot="MR180" display="off"/>
-<attribute name="POPULARITY" value="11" x="17.78" y="17.4625" size="1.778" layer="28" rot="MR180" display="off"/>
 <attribute name="VALUE" x="10.16" y="18.0975" size="1.778" layer="28" ratio="10" rot="MR180"/>
 </element>
@@
 </element>
 <element name="X2" library="con-amp-micro-mate-n-lock" package="4-794618-2" value="2X6-A" x="36.195" y="24.765" smashed="yes" rot="R90">
-<attribute name="NAME" x="32.155" y="8.275" size="1.27" layer="25" rot="R90"/>
+<attribute name="NAME" x="34.15125" y="22.7725" size="0.8128" layer="25"/>
 </element>
 <element name="RS" library="testpad" library_urn="urn:adsk.eagle:library:385" package="B1,27" package3d_urn="urn:adsk.eagle:package:27944/2" value="PTR1B1,27" x="25.0825" y="20.1676" smashed="yes" rot="MR0">
@@
 <contactref element="C6" pad="2"/>
 <contactref element="IC1" pad="5"/>
-<contactref element="IC1" pad="21"/>
 <contactref element="DA1" pad="8"/>
 <contactref element="DA1" pad="2"/>
@@
 </polygonfilldetails>
 </polygonpour>
+<contactref element="IC1" pad="21"/>
 </signal>
 <signal name="VCC">
