File: V2.x/Servo/LOCO-Servo.sch (EAGLE design)
At the start: 49 parts, among them IC1 Atmega 328-P, IC2 MCP2515, IC3 LM340MP-05, Q1 8MHz, Q2 16MHz, X2 2X6-A

Commit message: design clean up
Parts:
- IC1: device atmel:MEGA8-AI -> atmel:MEGA8
Other:
- note added: "Loco-Servo V2.2"
- note removed: "LOCO-Servo V2.1b-s"
- moved on the sheet: +5V, C11, C12, C13, C14, C15, C16, D1, D2, D3, D4, PLS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
